Commit message: Re-run onshape-to-robot, add Jetson motor test/tuning tools, and prep custom ODrive firmware build
- Re-export CAD assets and robot.urdf after onshape design edits
- Add web-based motor test/tuning UI (velocity and position control) and PID tuning script
- Add ESP32 USB<->UART bridge firmware for MKS xDrive Mini
- Fix ENCODER_CALIB_RANGE in setup_odrive.py (was 500x looser than firmware default,
  silently let bad encoder offset calibrations pass)
- Add setup_odrive_056.py, ported to the v0.5.2+ property renames, for testing
  against a custom-built v0.5.6 firmware (bad commutation on the stock v0.5.1
  MKS firmware traced to its open-loop, non-feedback offset calibration scan)

File: javis/robot.urdf (robot description, URDF)
Before this commit: robot javis, 3 links, 2 joints
Links:
- link body: geometry collision mesh filename=package://assets/16_copper.stl; collision mesh filename=package://assets/16_copper.stl
Joints:
- joint left_wheel: origin xyz=-0 -0.126 0.09295 rpy=1.5708 -0 3.14159 -> xyz=-0 -0.129 0.09295 rpy=1.5708 -0 3.14159
- joint right_wheel: origin xyz=-0 0.126 0.09295 rpy=1.5708 0 0 -> xyz=-0 0.129 0.09295 rpy=1.5708 0 0
