Commit message: Pull updated Onshape CAD and propagate through the sim
Wheel drivetrain redesigned: the gearbox/coupler/wheelconnector power
train is replaced by a direct-drive encoder/magnet mount, and link
names changed body/wheel/wheel_2 -> base_link/wheel_left/wheel_right.

- robot_constants.py: new link/geom names, wheel half-track 129->100mm,
  updated IMU/D435 mount positions.
- mass_model.py: GROUP_PATTERNS updated for the new/removed meshes;
  printed-part nominal mass replaced with a real 2026-08-12 weighing
  (1332.26 g, was a density-scaled guess); mass moment cache bumped.
- Fixed hardcoded old body-name references across velocity_task.py,
  bench_test_wheel.py, mdp/actions.py, mdp/events.py, inspect_mass.py,
  tune_sim_gains.py -- two of these (nominal_masses("wheel") /
  fuse_nominal("wheel")) were latent KeyError bugs that only happened
  to work before because the old left-wheel body was coincidentally
  named "wheel".
- Removed 17 orphaned mesh files no longer referenced by robot.urdf.

Verified: 32/32 mass-model checks pass, compiled MuJoCo model matches
the analytic model exactly (0.00e+00 error), all three tasks
(Javis-Payload-Flat/Rough, Javis-Velocity-Flat) build and smoke-train
cleanly. Existing checkpoints are stale against the new geometry and
need retraining.

Co-Authored-By: Claude Sonnet 5 <noreply@anthropic.com>

File: javis/robot.urdf (robot description, URDF)
Before this commit: robot javis, 3 links, 2 joints
Links:
- removed link body
- removed link wheel
- removed link wheel_2
- added link base_link, mass 1e-09; collision mesh filename=package://assets/16_copper.stl; collision mesh filename=package://assets/16_copper.stl
- added link wheel_left, mass 1e-09; collision mesh filename=package://assets/wheel_left.stl; visual mesh filename=package://assets/wheel_left.stl
- added link wheel_right, mass 1e-09; collision mesh filename=package://assets/wheel_right.stl; visual mesh filename=package://assets/wheel_right.stl
Joints:
- joint left_wheel: child wheel -> wheel_left; origin xyz=-0 -0.129 0.09295 rpy=1.5708 -0 3.14159 -> xyz=0 0.1 0.03 rpy=-1.5708 -0 -3.14159; parent body -> base_link
- joint right_wheel: child wheel_2 -> wheel_right; origin xyz=-0 0.129 0.09295 rpy=1.5708 0 0 -> xyz=0 -0.1 0.03 rpy=1.5708 -0 -3.14159; parent body -> base_link
